File: Mitchel_Ezekiel_Robot/_autosave-Mitchel_Ezekiel_Robot.kicad_pcb (KiCad board)
At the start: 2 copper layers, 138.9 x 83.3 mm, 33 parts, among them J1 JTAG, J2 GPS MODULE, J3 Barrel_Jack_Switch, J4 Conn_01x06, J5 Conn_01x06, J6 Conn_01x04, J7 Conn_02x03_Odd_Even, Q1 SFH300, SW1 SW_SPST, U1 ESP32-DEVKITC-32E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

Commit message: Add robot outline footprint to PCB design
Added the 'Basic-Robot-Outline_1' footprint to Mitchel_Ezekiel_Robot.kicad_pcb, including edge cuts and fabrication details. Updated backup files to reflect the latest PCB changes and removed outdated backups.
Parts:
- moved D1 206.6 mm to (45.7, 275.1)
- moved J2 206.6 mm to (52.2, 274.7)
- moved Q1 206.6 mm to (5.85, 303.7)
- moved C3 206.6 mm to (37.4, 282.5)
- moved C4 206.6 mm to (37.4, 286.5)
- moved D4 206.6 mm to (45.7, 286.0)
- moved D6 206.6 mm to (45.7, 297.0)
- moved J3 206.6 mm to (-18.9, 294.5)
- moved R3 206.6 mm to (56.5, 282.5)
- moved R4 206.6 mm to (56.5, 286.5)
- moved C1 206.6 mm to (37.4, 274.4)
- moved C5 206.6 mm to (37.4, 290.6)
- moved C6 206.6 mm to (37.4, 294.6)
- moved C7 206.6 mm to (37.4, 298.7)
- moved D2 206.6 mm to (5.85, 296.2)
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Other:
- outline, holes or cut-outs redrawn
