File: Mitchel_Ezekiel_Robot/Mitchel_Ezekiel_Robot.kicad_pcb (KiCad board)
At the start: 2 copper layers, 138.9 x 83.3 mm, 33 parts, among them J1 JTAG, J2 GPS MODULE, J3 Barrel_Jack_Switch, J4 Conn_01x06, J5 Conn_01x06, J6 Conn_01x04, J7 Conn_02x03_Odd_Even, Q1 SFH300, SW1 SW_SPST, U1 ESP32-DEVKITC-32E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

Commit message: Update PCB layout and add new backup files
Added four new backup ZIP files. Updated component placements and properties in Mitchel_Ezekiel_Robot.kicad_pcb, including changes to footprints, positions, and silkscreen details. Removed autosave and lock files.
Parts:
- U3: value L293D -> Motor Driver
- moved Q1 151.2 mm to (207.1, 83.1), turned to -90 degrees
- moved D2 149.9 mm to (207.1, 91.0), turned to -90 degrees
- moved U3 142.5 mm to (160.3, 92.8), turned to 90 degrees
- moved J6 111.0 mm to (189.2, 86.0)
- moved C7 105.1 mm to (193.5, 88.2)
- moved D5 100.0 mm to (194.8, 70.0)
- moved D6 98.6 mm to (194.8, 110.1)
- moved C6 96.4 mm to (184.4, 81.5)
- moved C3 94.3 mm to (182.7, 91.6), turned to 90 degrees
- moved R2 88.3 mm to (194.9, 93.7)
- moved R5 87.2 mm to (194.9, 98.2)
- moved R3 87.1 mm to (195.0, 83.1)
- moved C5 83.9 mm to (172.3, 81.7), turned to 180 degrees
- moved C4 79.1 mm to (167.3, 96.7)
- moved C1 61.9 mm to (150.6, 78.7), turned to -90 degrees
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Other:
- outline, holes or cut-outs redrawn

Commit message: gerber complete -- maybe...
Parts:
- moved D3 4.00 mm to (81.2, 60.0)
- moved D1 0.13 mm to (86.6, 125.2)
- moved D4 0.13 mm to (81.0, 125.1)
Routing:
- net GND: track 0.00 -> 257.2 mm
- net +3V3: track 0.00 -> 202.5 mm
- net /ECHO: track 0.00 -> 141.9 mm
- net +BATT: track 0.00 -> 132.5 mm
- net /TRIG: track 0.00 -> 124.0 mm
- net /LMOTOR_3A: track 0.00 -> 110.0 mm
- net /REARLAMPS: track 0.00 -> 103.8 mm
- net /LMOTOR_4A: track 0.00 -> 102.1 mm
- net /LPWM_3A4A: track 0.00 -> 100.5 mm
- net /RMOTOR_2A: track 0.00 -> 99.8 mm
- net /RPWM_1A2A: track 0.00 -> 99.8 mm
- net /LENCODER_B: track 0.00 -> 78.4 mm
- net /RMOTOR_1A: track 0.00 -> 76.6 mm
- net /LENCODER_A: track 0.00 -> 72.9 mm
- net Net-(D3-K): track 0.00 -> 66.9 mm
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
Commit message: done
Routing:
- net +BATT: track 132.5 -> 292.7 mm
- net /RENCODER_A: track 0.00 -> 130.4 mm
- net /FRONTLAMPS: track 42.0 -> 161.4 mm
- net GND: track 257.2 -> 286.3 mm
- net /LMOTOR_4A: track 102.1 -> 101.3 mm

Commit message: pcb stage + images
Parts:
- U3: value Motor Driver -> L293D
- moved Q1 0.85 mm to (206.3, 83.0)
- moved D2 0.84 mm to (206.3, 91.0)
Routing:
- net +BATT: track 292.7 -> 0.00 mm
- net GND: track 286.3 -> 0.00 mm
- net +3V3: track 202.5 -> 0.00 mm
- net /FRONTLAMPS: track 161.4 -> 0.00 mm
- net /ECHO: track 141.9 -> 0.00 mm
- net /RENCODER_A: track 130.4 -> 0.00 mm
- net /TRIG: track 124.0 -> 0.00 mm
- net /LMOTOR_3A: track 110.0 -> 0.00 mm
- net /REARLAMPS: track 103.8 -> 0.00 mm
- net /LMOTOR_4A: track 101.3 -> 0.00 mm
- net /LENCODER_B: track 78.4 -> 0.00 mm
- net /LENCODER_A: track 72.9 -> 0.00 mm
- net Net-(D3-K): track 66.9 -> 0.00 mm
- net /JTAG_MTDO: track 43.2 -> 0.00 mm
- net Net-(D5-K): track 41.1 -> 0.00 mm
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- added copper zone on B.Cu, net GND

Commit message: pcb edit
Routing:
- net /LPWM_3A4A: track 83.1 -> 0.00 mm
- net /RMOTOR_2A: track 79.7 -> 0.00 mm
- net Net-(D5-K): track 0.00 -> 72.2 mm
- net /RPWM_1A2A: track 71.1 -> 0.00 mm
- net /RMOTOR_1A: track 68.0 -> 0.00 mm
- net /FRONTLAMPS: track 0.00 -> 48.9 mm
- net +BATT: track 0.00 -> 30.9 mm
- net +3V3: track 0.00 -> 27.6 mm
- net Net-(J4-Pin_2): track 0.00 -> 17.7 mm
- net Net-(D2-A): track 0.00 -> 8.92 mm
- net /PHOTOTRANS: track 0.00 -> 8.79 mm
- net Net-(J4-Pin_1): track 21.3 -> 23.6 mm

Commit message: readme update
Parts:
- moved J7 0.50 mm to (108.5, 108.8), turned to 180 degrees
Routing:
- net +3V3: track 27.6 -> 242.8 mm
- net /RPWM_1A2A: track 0.00 -> 192.7 mm
- net +BATT: track 30.9 -> 202.4 mm
- net /RENCODER_A: track 0.00 -> 135.0 mm
- net /TRIG: track 0.00 -> 127.6 mm
- net /FRONTLAMPS: track 48.9 -> 169.8 mm
- net /REARLAMPS: track 0.00 -> 119.5 mm
- net /ECHO: track 0.00 -> 115.4 mm
- net /PHOTOTRANS: track 8.79 -> 121.3 mm
- net /RENCODER_B: track 0.00 -> 111.3 mm
- net /LMOTOR_3A: track 0.00 -> 107.8 mm
- net /LMOTOR_4A: track 0.00 -> 92.7 mm
- net /LPWM_3A4A: track 0.00 -> 91.4 mm
- net Net-(D3-K): track 0.00 -> 89.2 mm
- net /RMOTOR_2A: track 0.00 -> 85.5 mm
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
Commit message: pcb edit
Routing:
- net GND: track 0.00 -> 23.3 mm
- net /RENCODER_B: track 111.3 -> 123.0 mm
- net /JTAG_MTCK: track 12.9 -> 19.1 mm
- net /TRIG: track 127.6 -> 132.9 mm
- net /JTAG_MTDO: track 53.9 -> 59.0 mm
- net /JTAG_MTDI: track 26.8 -> 31.0 mm
- net /JTAG_MTMS: track 15.0 -> 17.8 mm
- net +3V3: track 242.8 -> 244.9 mm
- net /PHOTOTRANS: track 121.3 -> 120.4 mm
- net Net-(D3-K): track 89.2 -> 89.9 mm
- net +BATT: track 202.4 -> 203.1 mm
