File: Mitchel_Ezekiel_Robot/Mitchel_Ezekiel_Robot.kicad_pcb (KiCad board)
At the start: 2 copper layers, 138.9 x 83.3 mm, 34 parts, among them J1 JTAG, J2 GPS MODULE, J3 Barrel_Jack_Switch, J4 Conn_01x06, J5 Conn_01x06, J6 Conn_01x04, J7 Conn_02x03_Odd_Even, Q1 SFH300, SW1 SW_SPST, U1 ESP32-DEVKITC-32E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

Commit message: pcb edit
Routing:
- net /JTAG_MTDO: track 58.3 -> 68.8 mm
- net /RENCODER_B: track 172.9 -> 177.8 mm
- net +BATT: track 511.8 -> 513.9 mm
- net /REARLAMPS: track 121.9 -> 121.1 mm
